Commit message: added an imu

File: description/cubesat.urdf.xacro (robot description, xacro)
@@ -3,3 +3,4 @@
     <xacro:include filename="gazebo_control.xacro"/>
     <xacro:include filename="cubesat_core.xacro"/>
+    <xacro:include filename="imu.xacro"/>
 </robot>

File: description/cubesat_core.xacro (robot description, xacro)
@@ -51,5 +51,5 @@
     </link>
                <gazebo reference = 'sat_body'>
-                <material>Gazebo/SkyBlue </material>
+                <material>Gazebo/Orange </material>
             </gazebo>
     <!-- reaction_wheel_xz link (lettering referes to the plane parallel to them) -->
@@ -77,5 +77,5 @@
     </link>
              <gazebo reference = 'rec_wheel_xz'>
-                <material>Gazebo/Black</material>
+                <material>Gazebo/Motorway</material>
             </gazebo>
     <!-- reaction wheel in yz plane link -->
@@ -83,5 +83,5 @@
         <parent link="sat_body" />
         <child link="rec_wheel_yz" />
-        <origin xyz="0.05 0.0 0.0" rpy="0 -${pi/2} 0" />
+        <origin xyz="0.05 0.0 0.0" rpy="0 ${pi/2} 0" />
         <axis xyz="0.0 0.0 1.0" />
     </joint>
@@ -103,5 +103,5 @@
     </link>
              <gazebo reference = 'rec_wheel_yz'>
-                <material>Gazebo/Black</material>
+                <material>Gazebo/Motorway</material>
             </gazebo>
     <!-- reaction wheel in xy plane link -->
@@ -109,5 +109,5 @@
         <parent link="sat_body" />
         <child link="rec_wheel_xy" />
-        <origin xyz="0.0 0.0 -0.15" rpy="0 0 0" />
+        <origin xyz="0.0 0.0 -0.15" rpy="0 ${pi} 0" />
         <axis xyz="0.0 0.0 1.0" />
     </joint>
@@ -129,5 +129,5 @@
     </link>
              <gazebo reference = 'rec_wheel_xy'>
-                <material>Gazebo/Black</material>
+                <material>Gazebo/Motorway</material>
             </gazebo>
 </robot>

File: description/gazebo_control.xacro (robot description, xacro)
@@ -1,53 +1,21 @@
 <?xml version="1.0"?>
-<robot xmlns:xacro="http://www.ros.org/wiki/xacro">
-    <!-- Gazebo ROS 2 Control Plugin -->
-    <gazebo>
-        <plugin name="gazebo_ros2_control" filename="libgazebo_ros2_control.so"/>
-    </gazebo>
-    <!-- Reaction Wheel X -->
-    <gazebo>
-        <plugin name="rw_x_controller" filename="libgazebo_ros2_control.so">
-            <joint>rw_x_joint</joint>
-        </plugin>
-    </gazebo>
-    <!-- Reaction Wheel Y -->
-    <gazebo>
-        <plugin name="rw_y_controller" filename="libgazebo_ros2_control.so">
-            <joint>rw_y_joint</joint>
-        </plugin>
-    </gazebo>
-    <!-- Reaction Wheel Z -->
-    <gazebo>
-        <plugin name="rw_z_controller" filename="libgazebo_ros2_control.so">
-            <joint>rw_z_joint</joint>
-        </plugin>
-    </gazebo>
-    <!-- Transmission Setup -->
-    <transmission name="rw_x_trans">
-        <type>transmission_interface/SimpleTransmission</type>
-        <joint name="rw_x_joint">
-            <hardwareInterface>effort_controllers/JointEffortController</hardwareInterface>
-        </joint>
-        <actuator name="rw_x_motor">
-            <hardwareInterface>effort_controllers/JointEffortController</hardwareInterface>
-        </actuator>
-    </transmission>
-    <transmission name="rw_y_trans">
-        <type>transmission_interface/SimpleTransmission</type>
-        <joint name="rw_y_joint">
-            <hardwareInterface>effort_controllers/JointEffortController</hardwareInterface>
-        </joint>
-        <actuator name="rw_y_motor">
-            <hardwareInterface>effort_controllers/JointEffortController</hardwareInterface>
-        </actuator>
-    </transmission>
-    <transmission name="rw_z_trans">
-        <type>transmission_interface/SimpleTransmission</type>
-        <joint name="rw_z_joint">
-            <hardwareInterface>effort_controllers/JointEffortController</hardwareInterface>
-        </joint>
-        <actuator name="rw_z_motor">
-            <hardwareInterface>effort_controllers/JointEffortController</hardwareInterface>
-        </actuator>
-    </transmission>
+<robot xmlns:xacro="http://www.ros.org/wiki/xacro" >
+	<gazebo>
+	<plugin name="front_wheel" filename="libgazebo_ros_diff_drive.so">
+    	<!-- Wheel Information -->
+        <left_joint>rec_wheel_xz_joint</left_joint>
+        <right_joint>rec_wheel_yz_joint</right_joint>
+        <wheel_separation>0.35</wheel_separation>
+        <wheel_diameter>0.1</wheel_diameter>
+        <!-- Limit -->
+        <max_wheel_torque>200</max_wheel_torque>
+        <max_wheel_acceleration>10.0</max_wheel_acceleration>
+        <!-- Output -->
+        <odometry_frame>odom</odometry_frame>
+        <robot_base_frame>base_link</robot_base_frame>
+        <publish_odom>true</publish_odom>
+        <publish_odom_tf>true</publish_odom_tf>
+        <publish_wheel_tf>true</publish_wheel_tf>
+	</plugin>
+  	</gazebo>
 </robot>

Commit message: world camera position updated, and succssfully applied basic custom plugins

File: description/cubesat.urdf.xacro (robot description, xacro)
@@ -1,6 +1,6 @@
 <?xml version="1.0"?>
 <robot xmlns:xacro="http://www.ros.org/wiki/xacro"  name="robot">
-    <xacro:include filename="gazebo_control.xacro"/>
+    <!-- <xacro:include filename="gazebo_control.xacro"/> -->
     <xacro:include filename="cubesat_core.xacro"/>
-    <xacro:include filename="imu.xacro"/>
+    <!-- <xacro:include filename="imu.xacro"/> -->
 </robot>

File: description/cubesat_core.xacro (robot description, xacro)
@@ -2,7 +2,12 @@
 <robot xmlns:xacro="http://www.ros.org/wiki/xacro">
     <xacro:include filename="inertial_macros.xacro" />
-<!-- adding the variable -->
-    <xacro:property name="wheel_radius" value="0.05"/>
-    <xacro:property name="wheel_thick" value="0.04"/>
+<gazebo>
+    <plugin name="my_model_plugin" filename="libmy_model_plugin.so">
+        <model_vel>0.2</model_vel>
+    </plugin>
+</gazebo>
+    <!-- adding the variable -->
+    <xacro:property name="wheel_radius" value="0.05" />
+    <xacro:property name="wheel_thick" value="0.04" />
     <material name="white">
         <color rgba="1.0 1.0 1.0 1.0" />
@@ -21,7 +26,7 @@
     <!-- base_footprint link -->
     <joint name="base_footprint_joint" type="fixed">
-        <parent link="base_link"/>
-        <child link="base_footprint"/>
-        <origin xyz="0.0 0.0 0.0" rpy="0.0 0.0 0.0"/>
+        <parent link="base_link" />
+        <child link="base_footprint" />
+        <origin xyz="0.0 0.0 0.0" rpy="0.0 0.0 0.0" />
     </joint>
     <link name="base_footprint"></link>
@@ -50,7 +55,7 @@
         </xacro:inertial_box>
     </link>
-               <gazebo reference = 'sat_body'>
-                <material>Gazebo/Orange </material>
-            </gazebo>
+    <gazebo reference='sat_body'>
+        <material>Gazebo/Orange </material>
+    </gazebo>
     <!-- reaction_wheel_xz link (lettering referes to the plane parallel to them) -->
     <joint name="rec_wheel_xz_joint" type="continuous">
@@ -76,7 +81,7 @@
         </xacro:inertial_cylinder>
     </link>
-             <gazebo reference = 'rec_wheel_xz'>
-                <material>Gazebo/Motorway</material>
-            </gazebo>
+    <gazebo reference='rec_wheel_xz'>
+        <material>Gazebo/Motorway</material>
+    </gazebo>
     <!-- reaction wheel in yz plane link -->
     <joint name="rec_wheel_yz_joint" type="continuous">
@@ -102,7 +107,7 @@
         </xacro:inertial_cylinder>
     </link>
-             <gazebo reference = 'rec_wheel_yz'>
-                <material>Gazebo/Motorway</material>
-            </gazebo>
+    <gazebo reference='rec_wheel_yz'>
+        <material>Gazebo/Motorway</material>
+    </gazebo>
     <!-- reaction wheel in xy plane link -->
     <joint name="rec_wheel_xy_joint" type="continuous">
@@ -128,6 +133,6 @@
         </xacro:inertial_cylinder>
     </link>
-             <gazebo reference = 'rec_wheel_xy'>
-                <material>Gazebo/Motorway</material>
-            </gazebo>
+    <gazebo reference='rec_wheel_xy'>
+        <material>Gazebo/Motorway</material>
+    </gazebo>
 </robot>

File: description/imu.xacro (robot description, xacro)
@@ -4,13 +4,7 @@
         <parent link="sat_body" />
         <child link="imu_link" />
-        <origin xyz="0.605 0.0 0.08" rpy="0.0 0.0 0.0" />
+        <origin xyz="0.0 0.0 0.00" rpy="0.0 0.0 0.0" />
     </joint>
     <link name="imu_link">
-        <visual>
-            <geometry>
-                <box size="0.01 0.03 0.03" />
-                <material name="white" />
-            </geometry>
-        </visual>
     </link>
   <gazebo reference="imu_link">
@@ -25,5 +19,4 @@
         <bodyName>imu_link</bodyName>
         <updateRateHZ>10.0</updateRateHZ>
-        <gaussianNoise>0.1</gaussianNoise>
         <xyzOffset>0 0 0</xyzOffset>
         <rpyOffset>0 0 0</rpyOffset>
